File: PCB/PCB/PCB.kicad_sch (KiCad schematic)
At the start: 3 parts, among them M1 Motor_Servo, U1 NodeMCU_1.0_(ESP-12E), U2 DS18B20

Commit message: version 1.01
Parts:
- removed U2: DS18B20, Package_TO_SOT_THT:TO-92_Inline, symbol Sensor_Temperature:DS18B20
- added R1: 4.7K, Resistor_THT:R_Axial_DIN0204_L3.6mm_D1.6mm_P5.08mm_Horizontal, symbol Device:R
- added U2: HC-SR04, HC-SR04(1):XCVR_HC-SR04, symbol HC-SR04:HC-SR04
- added U3: DS18B20, Package_TO_SOT_THT:TO-92_Inline, symbol Sensor_Temperature:DS18B20
- M1: footprint Connector_PinHeader_1.27mm:PinHeader_1x03_P1.27mm_Vertical -> Connector_PinHeader_2.00mm:PinHeader_1x03_P2.00mm_Vertical
Connections:
- net at M1.2 (+): now also U1.16 (3.3V); no longer U1.25 (3.3V)
- net at U1.28 (D2(GPIO4)): now also U2.3 (ECHO)
- net at M1.3 (-): now also U1.17 (GND); no longer U1.24 (GND)
- net at U1.10 (GND): now also U3.1 (GND)
- net at U1.11 (3.3V): now also R1.1, U3.3 (V_{DD})
- net at U1.20 (D8(GPIO15)): now also M1.1 (PWM)
- net at U1.21 (D7(GPIO13)): now also R1.2, U3.2 (DQ)
- net at U1.27 (D3(GPIO0)): now also U2.2 (TRIG)
- net at U1.29 (D1(GPIO5)): no longer M1.1 (PWM)
- new net: U1.24 (GND), U2.4 (GND)
- new net: U1.25 (3.3V), U2.1 (VCC)
